File: PCBs/testboard/V2/testboard_v2.kicad_sch (KiCad schematic)
At the start: 29 parts, among them J1 FLEX pin1, J10 Conn_01x01, J11 Conn_01x01, J12 Conn_01x01, J13 Conn_01x02_Socket, J2 FLEX pin2, J3 FSR pin2, J4 FSR pin1, J5 Conn_01x02_Socket, J9 Conn_01x01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

Commit message: V2 updated for USB
Parts:
- added C11: 22uF, Capacitor_SMD:C_0603_1608Metric_Pad1.08x0.95mm_HandSolder, symbol Device:C
- added C12: 10uF, Capacitor_SMD:C_0603_1608Metric_Pad1.08x0.95mm_HandSolder, symbol Device:C
- added C13: 0.1uF, Capacitor_SMD:C_0603_1608Metric_Pad1.08x0.95mm_HandSolder, symbol Device:C
- added J6: USB_Conn, Connector_PinHeader_2.54mm:PinHeader_1x04_P2.54mm_Vertical, symbol Connector_Generic:Conn_01x04
- added U1: LD1117S33TR_SOT223, Package_TO_SOT_SMD:SOT-223-3_TabPin2, symbol Regulator_Linear:LD1117S33TR_SOT223
- added Y1: MAX7375AXR805, Package_TO_SOT_SMD:SOT-323_SC-70, symbol Oscillator:MAX7375AXR805
Connections:
- net DEBUG_1: now also U2.41 (PA8); no longer U2.42 (PA9)
- net GND: now also C11.2, C12.2, C13.2, J6.4 (Pin_4), U1.1 (GND), Y1.3 (GND)
- net VCC: now also C11.1, C13.1, U1.2 (VO), Y1.1 (V+)
- net USB_D-: now reaches U2.44 (PA11)
- net USB_D-: now also J6.2 (Pin_2)
- net USB_D+: now reaches U2.45 (PA12)
- net USB_D+: now also J6.3 (Pin_3)
- net PH0: now reaches U2.5 (PH0)
- net PH0: now also Y1.2 (CLOCK)
- new net USB_VBUS_5V: C12.1, J6.1 (Pin_1), U1.3 (VI), U2.42 (PA9)
- no-connect marks 41 -> 37
Other:
- note added: "Crystal oscillator SHOULD BE PLACED NEXT TO MCU AWAY FROM DATA LINES"
- note added: "Regulator for USB power"

Commit message: V2 schematic done - awaiting layout from kenobi
Parts:
- added R1, R2: 22 Ohm, Capacitor_SMD:C_0603_1608Metric_Pad1.08x0.95mm_HandSolder, symbol Device:R
Connections:
- net USB_D+: now also R2.1; no longer J6.3 (Pin_3)
- net USB_D-: now also R1.1; no longer J6.2 (Pin_2)
- new net: J6.3 (Pin_3), R2.2
- new net: J6.2 (Pin_2), R1.2
Other:
- moved on the sheet: J6
