File: PCBs/finalboard/V1/finalboard_v1.kicad_sch (KiCad schematic)
At the start: 45 parts, among them J1 Conn_01x02_Socket, J10 Conn_01x01, J11 Conn_01x01, J12 Conn_01x01, J13 Conn_01x02_Socket, J2 Conn_01x02_Socket, J3 Conn_01x02_Socket, J4 Conn_01x02_Socket, J5 Conn_01x02_Socket, J6 USB_Conn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

Commit message: Finalboard-V1 layout done (by kenobi)
Connections:
- net USB+: now reaches J6.3 (Pin_3), R2.2
- net USB-: now reaches J6.2 (Pin_2), R1.2
Other:
- moved on the sheet: R1, R2
Changed lines of the file:
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@@
 	(wire
 		(pts
-			(xy 50.8 71.12) (xy 53.34 71.12)
+			(xy 33.02 71.12) (xy 35.56 71.12)
 		)
 		(stroke
@@
 	(wire
 		(pts
-			(xy 50.8 68.58) (xy 53.34 68.58)
+			(xy 33.02 68.58) (xy 35.56 68.58)
 		)
 		(stroke
@@
 	)
 	(label "USB_D-"
-		(at 50.8 68.58 180)
+		(at 33.02 68.58 180)
 		(effects
 			(font
@@
 	)
 	(label "USB_D+"
-		(at 50.8 71.12 180)
+		(at 33.02 71.12 180)
 		(effects
 			(font
@@
 		)
 	)
+	(label "USB+"
+		(at 60.96 71.12 180)
+		(effects
+			(font
+				(size 1.27 1.27)
+			)
+			(justify right bottom)
+		)
+	)
 	(label "FLEX_3-"
 		(at 66.04 124.46 180)
@@
 		)
 	)
+	(label "USB-"
+		(at 60.96 68.58 180)
+		(effects
+			(font
+				(size 1.27 1.27)
+			)
+			(justify right bottom)
+		)
+	)
 	(label "VCC"
 		(at 168.91 180.34 0)
@@
 		)
 	)
+	(label "USB-"
+		(at 43.18 68.58 0)
+		(effects
+			(font
+				(size 1.27 1.27)
+			)
+			(justify left bottom)
+		)
+	)
 	(label "VCC"
 		(at 227.33 34.29 90)
@@
 		)
 	)
+	(label "USB+"
+		(at 43.18 71.12 0)
+		(effects
+			(font
+				(size 1.27 1.27)
+			)
+			(justify left bottom)
+		)
+	)
 	(label "USB_VBUS_5V"
 		(at 128.27 180.34 180)
@@
 	(symbol
 		(lib_id "Device:R")
-		(at 57.15 71.12 90)
+		(at 39.37 71.12 90)
 		(unit 1)
 		(exclude_from_sim no)
@@
 		(dnp no)
 		(property "Reference" "R2"
-			(at 52.832 73.152 90)
+			(at 35.052 73.152 90)
 			(effects
 				(font
@@
 		)
 		(property "Value" "22 Ohm"
-			(at 58.928 73.66 90)
+			(at 41.148 73.66 90)
 			(effects
 				(font
@@
 		)
 		(property "Footprint" "Resistor_SMD:R_0603_1608Metric_Pad0.98x0.95mm_HandSolder"
-			(at 57.15 72.898 90)
+			(at 39.37 72.898 90)
 			(effects
 				(font
@@
 		)
 		(property "Datasheet" "~"
-			(at 57.15 71.12 0)
+			(at 39.37 71.12 0)
 			(effects
 				(font
@@
 		)
 		(property "Description" "Resistor"
-			(at 57.15 71.12 0)
+			(at 39.37 71.12 0)
 			(effects
 				(font
@@
 	(symbol
 		(lib_id "Device:R")
-		(at 57.15 68.58 90)
+		(at 39.37 68.58 90)
 		(unit 1)
 		(exclude_from_sim no)
@@
 		(dnp no)
 		(property "Reference" "R1"
-			(at 52.578 66.802 90)
+			(at 34.798 66.802 90)
 			(effects
 				(font
@@
 		)
 		(property "Value" "22 Ohm"
-			(at 58.674 67.056 90)
+			(at 40.894 67.056 90)
 			(effects
 				(font
@@
 		)
 		(property "Footprint" "Resistor_SMD:R_0603_1608Metric_Pad0.98x0.95mm_HandSolder"
-			(at 57.15 70.358 90)
+			(at 39.37 70.358 90)
 			(effects
 				(font
@@
 		)
 		(property "Datasheet" "~"
-			(at 57.15 68.58 0)
+			(at 39.37 68.58 0)
 			(effects
 				(font
@@
 		)
 		(property "Description" "Resistor"
-			(at 57.15 68.58 0)
+			(at 39.37 68.58 0)
 			(effects
 				(font
