File: PCBs/finalboard/V2/finalboard_v2.kicad_pcb (KiCad board)
At the start: 2 copper layers, 60 x 60 mm, 45 parts, among them J1 Conn_01x02_Socket, J10 Conn_01x01, J11 Conn_01x01, J12 Conn_01x01, J13 Conn_01x02_Socket, J2 Conn_01x02_Socket, J3 Conn_01x02_Socket, J4 Conn_01x02_Socket, J5 Conn_01x02_Socket, J6 USB_Conn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

Commit message: Edit finalboard v2 to fix pinout on imu
Connections:
- U4 pad 13: unconnected-(U4-SCL-Pad13) -> /SPI_SCK
- U4 pad 14: unconnected-(U4-SDA-Pad14) -> /SPI_MOSI
- U4 pad 2: /SPI_MOSI -> unconnected-(U4-SDX-Pad2)
- U4 pad 3: /SPI_SCK -> unconnected-(U4-SCX-Pad3)
Routing:
- net /SPI_SCK: track 8.99 -> 1.30 mm
- net /SPI_MOSI: track 8.86 -> 5.69 mm
